File: mk1_better_pcb/master_teststand_v1.brd (EAGLE design)
At the start: 160 x 100 mm, 74 parts, among them Q1 FDN360P, Q10 FDN360P, Q2 FDN360P, Q3 FDN360P, Q4 FDN360P, Q5 FDN360P, Q6 FDN360P, Q7 FDN360P, Q8 FDN360P, Q9 FDN360P

Commit message: data collection
Parts:
- added X1, X10, X11, X12, X14, X15, X16, X2, X3, X4, X5, X6, X7, X8, X9: (no value), con-ptr500:AK300/2
- added X13: (no value), con-ptr500:AK300/3
Connections:
- new net ESTOP_SENSE1: X1.2
- new net ESTOP_SENSE2: X2.2
- new net ESTOP_SENSE3: X3.2
- new net ESTOP_SENSE4: X14.2
- new net ESTOP_SENSE5: X15.2
- new net ESTOP_SENSE6: X16.2
- new net N$21: X1.1
- new net N$22: X11.1
- new net N$23: X2.1
- new net N$24: X12.1
- new net N$25: X3.1
- new net N$26: X14.1
- new net N$27: X15.1
- new net N$28: X16.1
- new net N$31: X10.1
- new net N$33: X9.1
- new net N$37: X7.1
- new net N$39: X6.1
- new net N$41: X5.1
- new net N$43: X4.1
- net 12V: now also X10.2, X11.2
- net ESTOP_SENSE: now also X12.2
- net FUEL_VALVE: now also X5.2
- net GREEN: now also X13.1
- net IGN: now also X6.2
- net OUT1: now also X7.2
- net OUT2: now also X8.1, X8.2
- net OUT3: now also X9.2
- net OXYGEN_VALVE: now also X4.2
- net RED: now also X13.3
- net YELLOW: now also X13.2
