File: mk1_better_pcb/master_teststand_v1.sch (EAGLE design)
At the start: 1 part

Commit message: running hotfire
Parts:
- removed B1: ARDUINO_UNO_R3, SparkFun-Boards:ARDUINO_UNO_R3
- added R1: 100, SparkFun-Resistors:100OHM-0603-1/4W-5%
- added U$1: ESP32DEVKITV1, ESP32-DEVKITV1:ESP32DEVKITV1
Connections:
- new net DONT_USE: U$1.IO1, U$1.IO12, U$1.IO15, U$1.IO2, U$1.IO3, U$1.IO5
- new net FUEL_VALVE: U$1.IO22
- new net GND: R1.1, U$1.GND@1, U$1.GND@2
- new net GREEN_LIGHT_UC: U$1.IO21
- new net IGN_UC: U$1.IO4
- new net OUT1_UC: U$1.IO14
- new net OUT2_UC: U$1.IO13
- new net OXYGEN_VALVE: U$1.IO23
- new net RED_LIGHT_UC: U$1.IO18
- new net RX: U$1.IO16
- new net THERMORESISITOR1: U$1.IO25
- new net THERMORESISITOR2: U$1.IO26
- new net THERMORESISTOR3: U$1.IO27
- new net TRANSDUCER1: U$1.VP-OI36
- new net TRANSDUCER2: U$1.VN-IO39
- new net TRANSDUCER3: U$1.IO34
- new net TRANSDUCER4: U$1.IO35
- new net TRANSDUCER5: U$1.IO32
- new net TRANSDUCER6: U$1.IO33
- new net TX: U$1.IO17
- new net YELLOW_LIGHT_UC: U$1.IO19

Commit message: run1
Parts:
- added D1: RS1M, Diode:DIODE_RS1M_SMA
- added Q2: FDN360P, transistor-power:FDN360P
- added R10, R11: 10k, SparkFun-Resistors:10KOHM-0603-1/10W-1%
- added R12: 5.6k, SparkFun-Resistors:5.6KOHM-0603-1/10W-1%
- added R2, R3, R4, R5, R6: 150, SparkFun-Resistors:150OHM-0603-1/10W-1%
- added R7, R8, R9: 100k, SparkFun-Resistors:100KOHM-0603-1/10W-1%
- added T1: (no value), transistor-neu-to92:MMBT2222ALT1-NPN-SOT23-BEC
- R1: value 100 -> 150; device SparkFun-Resistors:100OHM-0603-1/4W-5% -> SparkFun-Resistors:150OHM-0603-1/10W-1%
Connections:
- net FUEL_VALVE renamed FUEL_VALVE_UC
- removed net THERMORESISITOR1: U$1.IO25
- removed net THERMORESISITOR2: U$1.IO26
- new net ESTOP_VCC: Q2.S, R11.2
- new net N$3: Q2.G, R11.1, T1.C
- new net N$5: R12.2, T1.B
- new net OXYGEN_VALVE_UC: R12.1, U$1.IO23
- new net THERMORESISTOR1: R7.2, U$1.IO25
- new net THERMORESISTOR2: R8.2, U$1.IO26
- net GND: now also D1.A, R10.1, R2.1, R3.1, R4.1, R5.1, R6.1, R7.1, R8.1, R9.1, T1.E
- net OXYGEN_VALVE: now also D1.C, Q2.D, R10.2; no longer U$1.IO23
- net THERMORESISTOR3: now also R9.2
- net TRANSDUCER1: now also R1.2
- net TRANSDUCER2: now also R2.2
- net TRANSDUCER3: now also R3.2
- net TRANSDUCER4: now also R4.2
- net TRANSDUCER5: now also R5.2
- net TRANSDUCER6: now also R6.2
Other:
- moved on the sheet: R1

Commit message: data collection
Parts:
- added D10, D2, D3, D4, D5, D6, D7, D8, D9: RS1M, Diode:DIODE_RS1M_SMA
- added Q1, Q10, Q3, Q4, Q5, Q6, Q7, Q8, Q9: FDN360P, transistor-power:FDN360P
- added R13, R14, R16, R17, R19, R20, R22, R23, R25, R26, R29, R30, R32, R33, R35, R36, R38, R39: 10k, SparkFun-Resistors:10KOHM-0603-1/10W-1%
- added R15, R18, R21, R24, R27, R31, R34, R37, R40, R41: 5.6k, SparkFun-Resistors:5.6KOHM-0603-1/10W-1%
- added R28: 150, SparkFun-Resistors:150OHM-0603-1/10W-1%
- added T10, T2, T3, T4, T5, T6, T7, T8, T9: (no value), transistor-neu-to92:MMBT2222ALT1-NPN-SOT23-BEC
- added U$2, U$3: DC-DC-STEP-DOWN-LM2596, 1484249208697-powermodules:DC-DC-STEP-DOWN-LM2596
- added X1, X10, X11, X12, X14, X15, X16, X2, X3, X4, X5, X6, X7, X8, X9: (no value), con-ptr500:AK300/2
- added X13: (no value), con-ptr500:AK300/3
Connections:
- removed net RX: U$1.IO16
- removed net TX: U$1.IO17
- new net 12V: Q10.S, Q7.S, Q8.S, Q9.S, R30.2, R33.2, R36.2, R39.2, U$3.OUT+, X10-2.KL, X11-2.KL
- new net 5V: U$1.VIN, U$2.OUT+
- new net ESTOP_SENSE: R31.1, R41.2, X12-2.KL
- new net ESTOP_SENSE1: X1-2.KL
- new net ESTOP_SENSE2: X2-2.KL
- new net ESTOP_SENSE3: X3-2.KL
- new net ESTOP_SENSE4: X14-2.KL
- new net ESTOP_SENSE5: X15-2.KL
- new net ESTOP_SENSE6: X16-2.KL
- new net FUEL_VALVE: D2.C, Q1.D, R13.2, X5-2.KL
- new net GREEN: D8.C, Q8.D, R32.2, X13-1.KL
- new net IGN: D3.C, Q3.D, R16.2, X6-2.KL
- new net LOADCELL: R28.2, U$1.IO4
- new net N$1: Q1.G, R14.1, T2.C
- new net N$10: R24.2, T5.B
- new net N$11: Q6.G, R26.1, T6.C
- new net N$12: R27.2, T6.B
- new net N$13: Q7.G, R30.1, T7.C
- new net N$14: R31.2, T7.B
- new net N$15: Q8.G, R33.1, T8.C
- new net N$16: R34.2, T8.B
- new net N$17: Q9.G, R36.1, T9.C
- new net N$18: R37.2, T9.B
- new net N$19: Q10.G, R39.1, T10.C
- new net N$2: R15.2, T2.B
- new net N$20: R40.2, T10.B
- new net N$21: X1-1.KL
- new net N$22: X11-1.KL
- new net N$23: X2-1.KL
- new net N$24: X12-1.KL
- new net N$25: X3-1.KL
- new net N$26: X14-1.KL
- new net N$27: X15-1.KL
- new net N$28: X16-1.KL
- new net N$31: X10-1.KL
- new net N$33: X9-1.KL
- new net N$37: X7-1.KL
- new net N$39: X6-1.KL
- new net N$4: Q3.G, R17.1, T3.C
- new net N$41: X5-1.KL
- new net N$43: X4-1.KL
- new net N$6: R18.2, T3.B
- new net N$7: Q4.G, R20.1, T4.C
- new net N$8: R21.2, T4.B
- new net N$9: Q5.G, R23.1, T5.C
- new net OUT1: D6.C, Q6.D, R25.2, X7-2.KL
- new net OUT2: D5.C, Q5.D, R22.2, X8-1.KL, X8-2.KL
- new net OUT3: D4.C, Q4.D, R19.2, X9-2.KL
- new net OUT3_UC: R21.1, U$1.IO16
- new net RED: D10.C, Q10.D, R38.2, X13-3.KL
- new net VCC: U$2.IN+, U$3.IN+
- new net YELLOW: D9.C, Q9.D, R35.2, X13-2.KL
- net ESTOP_VCC: now also D7.C, Q1.S, Q3.S, Q4.S, Q5.S, Q6.S, Q7.D, R14.2, R17.2, R20.2, R23.2, R26.2, R29.2
- net FUEL_VALVE_UC: now also R15.1
- net GND: now also D10.A, D2.A, D3.A, D4.A, D5.A, D6.A, D7.A, D8.A, D9.A, R13.1, R16.1, R19.1, R22.1, R25.1, R28.1, R29.1, R32.1, R35.1, R38.1, R41.1, T10.E, T2.E, T3.E, T4.E, T5.E, T6.E, T7.E, T8.E, T9.E, U$2.IN-, U$2.OUT-, U$3.IN-, U$3.OUT-
- net GREEN_LIGHT_UC: now also R34.1
- net IGN_UC: now also R18.1, U$1.IO17; no longer U$1.IO4
- net OUT1_UC: now also R27.1
- net OUT2_UC: now also R24.1
- net OXYGEN_VALVE: now also X4-2.KL
- net RED_LIGHT_UC: now also R40.1
- net YELLOW_LIGHT_UC: now also R37.1
Other:
- moved on the sheet: D1, Q2, R1, R10, R11, R12, R2, R3, R4, R5, R6, R7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
